File: Morse Mech.sch (KiCad schematic (older format))
At the start: 20 parts, among them P1 USB_OTG, P2 ICSP, SW1 Gateron Green, U1 EEPROM_SPI, Y1 16MHz

Commit message: Updated schematic with PTH crystal
Takes up less space than the SMD version, surprisingly...
Corresponding datasheet also updated.
Parts:
- Y1: footprint Crystals:Crystal_HC49-SD_SMD -> Crystals:Crystal_HC49-U_Vertical
Changed lines of the file:
@@
 F 0 "Y1" H 2650 4450 40  0000 C CNN
 F 1 "16MHz" H 2650 4150 40  0000 C CNN
-F 2 "Crystals:Crystal_HC49-SD_SMD" H 2650 4300 50  0001 C CNN
-F 3 "http://www.mouser.com/ds/2/741/LFXTAL003237Reel-940153.pdf" H 2650 4300 50  0001 C CNN
+F 2 "Crystals:Crystal_HC49-U_Vertical" H 2650 4300 50  0001 C CNN
+F 3 "http://www.mouser.com/ds/2/741/LFXTAL003240Bulk-940314.pdf" H 2650 4300 50  0001 C CNN
 	1    2650 4300
 	1    0    0    -1
